File: synthesizer/synthesizer.kicad_pcb (KiCad board)
At the start: 2 copper layers, 29.5 x 88.8 mm, 21 parts, among them SW1 SW_SOLO, SW2 SW_MUTE, SW3 SW_L, SW4 SW_R, U1 RaspberryPi_Pico

Commit message: Updated schematics
Parts:
- removed D1: GREEN, LED_THT:LED_D5.0mm
- removed SW4: SW_R, Button_Switch_THT:SW_PUSH_6mm
- added R1: 330Ω, Resistor_THT:R_Axial_DIN0207_L6.3mm_D2.5mm_P7.62mm_Horizontal, F.Cu at (103.1, 74.5)
- added R2: 330Ω, Resistor_THT:R_Axial_DIN0207_L6.3mm_D2.5mm_P7.62mm_Horizontal, F.Cu at (103.1, 77.8)
- added R3: 51Ω, Resistor_THT:R_Axial_DIN0207_L6.3mm_D2.5mm_P7.62mm_Horizontal, F.Cu at (125.4, 74.5)
- added R4: 51Ω, Resistor_THT:R_Axial_DIN0207_L6.3mm_D2.5mm_P7.62mm_Horizontal, F.Cu at (125.4, 77.8)
- added R5: 51Ω, Resistor_THT:R_Axial_DIN0207_L6.3mm_D2.5mm_P7.62mm_Horizontal, F.Cu at (125.4, 81.1)
- added R7: 330Ω, Resistor_THT:R_Axial_DIN0207_L6.3mm_D2.5mm_P7.62mm_Horizontal, F.Cu at (103.1, 81.1)
- added SW6: RotaryEncoder_Switch, Rotary_Encoder:RotaryEncoder_Bourns_Vertical_PEC12R-3xxxF-Sxxxx, F.Cu at (121.8, 93.5)
- SW1, SW2: footprint Button_Switch_THT:SW_PUSH_6mm -> Button_Switch_THT:SW_PUSH_6mm_H5mm
- SW3: value SW_L -> SW_PREV; footprint Button_Switch_THT:SW_PUSH_6mm -> Button_Switch_THT:SW_PUSH_6mm_H5mm
- U1: footprint Module_RaspberryPi_Pico:RaspberryPi_Pico_Common_THT_MountingHoles -> project_local:RPi_connector
- moved IN2 129.7 mm to (101.5, 114.9)
- moved OUT2 129.4 mm to (127.0, 115.0)
- moved VU5 126.1 mm to (112.5, 144.0)
- moved VU4 123.4 mm to (112.5, 137.5)
- moved VU3 121.5 mm to (112.5, 131.0)
- moved H1 118.0 mm to (101.8, 65.8)
- moved H2 118.0 mm to (126.7, 65.8)
- moved H3 118.0 mm to (101.8, 150.0)
- moved H4 118.0 mm to (126.7, 150.0)
- moved S1 118.0 mm to (114.2, 80.8)
- moved IN1 117.2 mm to (101.5, 131.5)
- moved OUT1 116.9 mm to (127.0, 131.4)
- moved SW2 113.2 mm to (123.0, 139.2), turned to -90 degrees
- moved SW1 112.4 mm to (123.0, 129.8), turned to -90 degrees
- moved VU2 112.2 mm to (112.5, 124.5)
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- renumbered PI1 to IN1, PI2 to IN2, PO1 to OUT1, PO2 to OUT2
Connections:
- net /LEFT_SW renamed /PREV_SW
- D2 pad 1: GND -> /R7D2
- D2 pad 2: Net-(D2-A) -> /MUTE_LED
- IN1 pad 6: /MUTE -> /MUTE_SIG
- IN2 pad 6: /MUTE -> /MUTE_SIG
- OUT1 pad 3: /I2S_OUT1_SD -> /I2S_OUT_SD
- OUT1 pad 4: /I2S_OUT1_SCK -> /I2S_OUT_SCK
- OUT1 pad 5: /I2S_OUT1_WS -> /I2S_OUT_WS
- OUT1 pad 6: /MUTE -> /MUTE_SIG
- OUT2 pad 3: /I2S_OUT2_SD -> /I2S_OUT_SD
- OUT2 pad 4: /I2S_OUT2_SCK -> /I2S_OUT_SCK
- OUT2 pad 5: /I2S_OUT2_WS -> /I2S_OUT_WS
- OUT2 pad 6: /MUTE -> /MUTE_SIG
- SW1 pad 2: /SOLO_SW -> /SOLO_BTN
- SW2 pad 2: /MUTE_SW -> /MUTE_BTN
- U1 pad 1: unconnected-(U1-GPIO0-Pad1) -> /MUTE_LED
- U1 pad 10: unconnected-(U1-GPIO7-Pad10) -> /I2S_IN2_SCK
- U1 pad 11: unconnected-(U1-GPIO8-Pad11) -> /I2S_IN2_WS
- U1 pad 12: unconnected-(U1-GPIO9-Pad12) -> /I2S_IN1_SD
- U1 pad 14: unconnected-(U1-GPIO10-Pad14) -> /I2S_IN1_SCK
- U1 pad 15: unconnected-(U1-GPIO11-Pad15) -> /I2S_IN1_WS
- U1 pad 16: unconnected-(U1-GPIO12-Pad16) -> /MUTE_BTN
- U1 pad 17: unconnected-(U1-GPIO13-Pad17) -> /I2S_OUT_SD
- U1 pad 19: unconnected-(U1-GPIO14-Pad19) -> /I2S_OUT_SCK
- U1 pad 20: unconnected-(U1-GPIO15-Pad20) -> /I2S_OUT_WS
- U1 pad 21: unconnected-(U1-GPIO16-Pad21) -> /VU_GREEN3
- U1 pad 22: unconnected-(U1-GPIO17-Pad22) -> /VU_GREEN2
- U1 pad 24: unconnected-(U1-GPIO18-Pad24) -> /VU_GREEN1
- U1 pad 25: unconnected-(U1-GPIO19-Pad25) -> /VU_YELLOW
- U1 pad 26: unconnected-(U1-GPIO20-Pad26) -> /VU_RED
- U1 pad 27: unconnected-(U1-GPIO21-Pad27) -> /SOLO_BTN
- U1 pad 29: unconnected-(U1-GPIO22-Pad29) -> /MUTE_SIG
- U1 pad 33: unconnected-(U1-AGND-Pad33) -> GND
- U1 pad 9: unconnected-(U1-GPIO6-Pad9) -> /I2S_IN2_SD
- VU1 pad 1: Net-(VU1-K) -> /VU_R1
- VU2 pad 1: Net-(VU1-K) -> /VU_R2
- VU3 pad 1: Net-(VU1-K) -> /VU_R3
- VU4 pad 1: Net-(VU1-K) -> /VU_R4
- VU5 pad 1: Net-(VU1-K) -> /VU_R5
Routing:
- added copper zone on B.Cu, net GND
Other:
- board text added: "2024.01"
- board text added: "3V"
- board text added: "CK"
- board text added: "Effects Module"
- board text added: "G"
- board text added: "GD"
- board text added: "M"
- board text added: "MT"
- board text added: "MUTE"
- board text added: "PREVIOUS"
- board text added: "R"
- board text added: "RPi"
- board text added: "SD"
- board text added: "SOLO"
- board text added: "VOLUME"
- board text added: "WS"
- board text added: "Y"
- board text added: "n0m1s"
- board text added: "v1.0"
