File: synthesizer/synthesizer.kicad_sch (KiCad schematic)
At the start: 27 parts, among them J1 Conn_02x20_Top_Bottom, J2 Conn_02x20_Top_Bottom, SW1 SW_SOLO, SW2 SW_MUTE, SW3 SW_L, SW4 SW_R, SW6 RotaryEncoder_Switch, U1 RaspberryPi_Pico

Commit message: Updated schematics
Parts:
- removed J1, J2: Conn_02x20_Top_Bottom, symbol Connector_Generic:Conn_02x20_Top_Bottom
- removed PI2: ~, project_local:PannelConnector, symbol project_local:PanelConnectorIn
- removed PO2: ~, project_local:PannelConnector, symbol project_local:PanelConnectorOut
- removed R1: 220Ω, symbol Device:R
- removed SW4: SW_R, Button_Switch_THT:SW_PUSH_6mm, symbol Switch:SW_Push
- added R2: 330Ω, Resistor_THT:R_Axial_DIN0207_L6.3mm_D2.5mm_P7.62mm_Horizontal, symbol Device:R
- added R3, R4, R5, R6: 51Ω, Resistor_THT:R_Axial_DIN0207_L6.3mm_D2.5mm_P7.62mm_Horizontal, symbol Device:R
- D1: value GREEN -> RED
- R1: renamed from R3; value 220Ω -> 330Ω; footprint (none) -> Resistor_THT:R_Axial_DIN0207_L6.3mm_D2.5mm_P7.62mm_Horizontal
- R7: renamed from R2; value 220Ω -> 330Ω; footprint (none) -> Resistor_THT:R_Axial_DIN0207_L6.3mm_D2.5mm_P7.62mm_Horizontal
- SW1, SW2: footprint Button_Switch_THT:SW_PUSH_6mm -> Button_Switch_THT:SW_PUSH_6mm_H5mm
- SW3: value SW_L -> SW_PREV; footprint Button_Switch_THT:SW_PUSH_6mm -> Button_Switch_THT:SW_PUSH_6mm_H5mm
- SW6: footprint (none) -> Rotary_Encoder:RotaryEncoder_Bourns_Vertical_PEC12R-3xxxF-Sxxxx
- U1: footprint Module_RaspberryPi_Pico:RaspberryPi_Pico_Common_THT_MountingHoles -> project_local:RPi_connector
- renumbered PI1 to IN1, PO1 to OUT1
Connections:
- net I2S_OUT1_SCK is gone; now on net I2S_OUT_SCK: OUT1.4 (SCK)
- net I2S_OUT1_SD is gone; now on net I2S_OUT_SD: OUT1.3 (SD)
- net I2S_OUT1_WS is gone; now on net I2S_OUT_WS: OUT1.5 (WS)
- net MUTE is gone; now on net MUTE_SIG: IN1.6 (MUTE), OUT1.6 (MUTE)
- net MUTE_SW is gone; now on net MUTE_BTN: SW2.2
- net SOLO_SW is gone; now on net SOLO_BTN: SW1.2
- net ENC_A: now also U1.31 (GPIO26_ADC0)
- net ENC_B: now also U1.34 (GPIO28_ADC2)
- net ENC_C: now also U1.32 (GPIO27_ADC1)
- net GND: now also R1.1, R7.1, U1.33 (AGND), R2.1, R3.1, R4.1, R5.1, R6.1; no longer D1.1 (K), D2.1 (K), R1.2
- net MUTE_LED: now also D2.2 (A), U1.9 (GPIO6); no longer R7.2
- net SCREEN_DC: now also U1.2 (GPIO1)
- net SCREEN_RES: now also U1.1 (GPIO0)
- net SCREEN_SPI_CLK: now also U1.5 (GPIO3)
- net SCREEN_SPI_CS: now also U1.4 (GPIO2)
- net SCREEN_SPI_MOSI: now also U1.6 (GPIO4)
- net SOLO_LED: now also D1.2 (A), U1.7 (GPIO5)
- net VU_GREEN1: now also U1.24 (GPIO18)
- net VU_GREEN2: now also U1.22 (GPIO17)
- net VU_GREEN3: now also U1.21 (GPIO16)
- net VU_RED: now also U1.26 (GPIO20)
- net VU_YELLOW: now also U1.25 (GPIO19)
- net I2S_IN_SD: now reaches U1.12 (GPIO9)
- net I2S_IN_SCK: now reaches U1.14 (GPIO10)
- net I2S_IN_WS: now reaches U1.15 (GPIO11)
- net MUTE_BTN: now reaches U1.16 (GPIO12)
- net I2S_OUT_SD: now reaches U1.17 (GPIO13)
- net I2S_OUT_SCK: now reaches U1.19 (GPIO14)
- net I2S_OUT_WS: now reaches U1.20 (GPIO15)
- net SOLO_BTN: now reaches U1.27 (GPIO21)
- net MUTE_SIG: now reaches U1.29 (GPIO22)
- net LEFT_SW renamed PREV_SW
- new net R6D1: D1.1 (K), R6.2
- new net R7D2: D2.1 (K), R7.2
- new net VU_R1: R1.2, VU1.1 (K)
- new net VU_R2: R2.2, VU2.1 (K)
- new net VU_R3: R3.2, VU3.1 (K)
- new net VU_R4: R4.2, VU4.1 (K)
- new net VU_R5: R5.2, VU5.1 (K)
- no-connect marks 0 -> 1
Other:
- note removed: "Secondary inter-panel connectors"
- moved on the sheet: D2, R1, R7, SW3, U1, VU1, VU2, VU3, VU4, VU5
